File: rp2040_stamp_console.kicad_pcb (KiCad board)
At the start: 2 copper layers, 36 x 53.7 mm, 37 parts, among them J1 USB_C_Receptacle_USB2.0, J2 Conn_Qwiic, SW1 SW_UP, SW2 SW_DOWN, SW3 SW_LEFT, SW4 SW_RIGHT, SW5 SW_A, SW6 SW_B, SW7 SW_POWER, U1 RP2040_Stamp

Commit message: Rev 2
Parts:
- removed kibuzzard-62C56D1C: G***, kibuzzard-62C56D1C
- added JP1: SJ_LOUDER, Jumper:SolderJumper-2_P1.3mm_Open_RoundedPad1.0x1.5mm, B.Cu at (123.0, 79.6)
- added kibuzzard-62DEDED4: G***, kibuzzard-62DEDED4, B.Cu at (116.7, 87.7)
- added kibuzzard-62DEDF00: G***, kibuzzard-62DEDF00, F.Cu at (117.8, 91.0)
- added kibuzzard-62DEDF0B: G***, kibuzzard-62DEDF0B, F.Cu at (117.8, 92.4)
- TP1, TP2: footprint TestPoint:TestPoint_Pad_2.0x2.0mm -> TestPoint:TestPoint_Pad_2.5x2.5mm
- turned D1 to 0 degrees
Connections:
- D1 pad 2: +3.3V -> Net-(D1-Pad2)
- D1 pad 3: Net-(D1-Pad3) -> +3.3V
- R1 pad 1: /LED_R -> /LED_B
- R1 pad 2: Net-(D1-Pad4) -> Net-(D1-Pad2)
- R2 pad 1: /LED_G -> /LED_R
- R2 pad 2: Net-(D1-Pad3) -> Net-(D1-Pad4)
- R3 pad 1: /LED_B -> /LED_G
- U1 pad 1: /LED_B -> /LED_G
- U1 pad 2: /LED_G -> /LED_R
- U1 pad 3: /LED_R -> /LED_B
- U1 pad 4: /SCL -> unconnected-(U1-Pad4)
- U1 pad 6: /LCD_CLK -> /SCL
- U1 pad 7: unconnected-(U1-Pad7) -> /LCD_CLK
Routing:
- net /SCL: track 24.8 -> 31.5 mm
- net Net-(D1-Pad4): track 2.08 -> 6.79 mm
- net /LED_B: track 22.0 -> 26.1 mm
- net Net-(D1-Pad3): track 3.91 -> 0.00 mm
- net /LED_R: track 26.1 -> 23.6 mm
- net Net-(D1-Pad2): track 0.00 -> 2.08 mm
- net Net-(D1-Pad1): track 7.55 -> 5.77 mm
- net /LED_G: track 23.6 -> 22.0 mm
- net +3.3V: track 38.5 -> 39.9 mm
- net /LCD_CLK: track 17.7 -> 18.5 mm
- net /SDA: track 26.1 -> 26.7 mm
- net /SPK-: track 41.5 -> 42.0 mm
- net GND: vias 53 -> 61
