File: rp2040_stamp_console.kicad_sch (KiCad schematic)
At the start: 26 parts, among them J1 USB_C_Receptacle_USB2.0, J2 Conn_Qwiic, SW1 SW_UP, SW2 SW_DOWN, SW3 SW_LEFT, SW4 SW_RIGHT, SW5 SW_A, SW6 SW_B, SW7 SW_POWER, U1 RP2040_Stamp

Commit message: Rev 2
Parts:
- added JP1: (no value), symbol Jumper:SolderJumper_2_Open
- C1: value 4.7uF -> (none); footprint Capacitor_SMD:C_0603_1608Metric -> (none)
- C2, C3, C4, C5: value 1uF -> (none); footprint Capacitor_SMD:C_0603_1608Metric -> (none)
- D1: value LED_BAGR -> (none); footprint LED_SMD_Extra:LED_RGBA_0606 -> (none); symbol Device:LED_BAGR -> Device:LED_GBAR
- DS1: value OLED-128O064D -> (none); footprint Display:OLED-128O064D -> (none)
- J1: value USB_C_Receptacle_USB2.0 -> (none); footprint Connector_USB:USB_C_Receptacle_HRO_TYPE-C-31-M-12 -> (none); LCSC (none) -> C165948
- J2: value Conn_Qwiic -> (none); footprint Connector_JST:JST_SH_SM04B-SRSS-TB_1x04-1MP_P1.00mm_Horizontal -> (none); LCSC (none) -> C145956
- LS1: value Speaker -> (none); footprint Buzzer_Beeper_Extra:CMT-5023S -> (none); LCSC (none) -> C94598
- R1, R2, R3: value 2K -> (none); footprint Resistor_SMD:R_0603_1608Metric -> (none)
- R4, R5: value 5.1K -> (none); footprint Resistor_SMD:R_0603_1608Metric -> (none)
- R6: value 390K -> (none); footprint Resistor_SMD:R_0603_1608Metric -> (none)
- SW1: value SW_UP -> (none); footprint Button_Switch_SMD_Extra:RMT-CZ66 -> (none); LCSC (none) -> C128939
- SW2: value SW_DOWN -> (none); footprint Button_Switch_SMD_Extra:RMT-CZ66 -> (none); LCSC (none) -> C128939
- SW3: value SW_LEFT -> (none); footprint Button_Switch_SMD_Extra:RMT-CZ66 -> (none); LCSC (none) -> C128939
- SW4: value SW_RIGHT -> (none); footprint Button_Switch_SMD_Extra:RMT-CZ66 -> (none); LCSC (none) -> C128939
- SW5: value SW_A -> (none); footprint Button_Switch_SMD_Extra:RMT-CZ66 -> (none); LCSC (none) -> C128939
- SW6: value SW_B -> (none); footprint Button_Switch_SMD_Extra:RMT-CZ66 -> (none); LCSC (none) -> C128939
- SW7: value SW_POWER -> (none); footprint Button_Switch_SMD:SW_SPDT_PCM12 -> (none); LCSC (none) -> C319020
- TP1: value TP_BATT+ -> (none); footprint TestPoint:TestPoint_Pad_2.0x2.0mm -> (none)
- TP2: value TP_BATT- -> (none); footprint TestPoint:TestPoint_Pad_2.0x2.0mm -> (none)
- U1: value RP2040_Stamp -> (none); footprint RP2040_Stamp:RP2040_Stamp_SMD -> (none)
Connections:
- net +3.3V: now also D1.3 (A); no longer D1.2 (A)
- net GND: now also JP1.2 (B)
- net LCD_CLK: now also U1.7 (GPIO6); no longer U1.6 (GPIO5)
- net LED_B: now also R1.1, U1.3 (GPIO2); no longer R3.1, U1.1 (GPIO0)
- net LED_G: now also R3.1, U1.1 (GPIO0); no longer R2.1, U1.2 (GPIO1)
- net LED_R: now also R2.1, U1.2 (GPIO1); no longer R1.1, U1.3 (GPIO2)
- net SCL: now also U1.6 (GPIO5); no longer U1.4 (GPIO3)
- net SPK-: now also JP1.1 (A)
- net at R1.2: now also D1.2 (BK); no longer D1.4 (RK)
- net at R2.2: now also D1.4 (RK); no longer D1.3 (GK)
Other:
- moved on the sheet: D1, LS1, R1, R2, R3
